Commit message: requirements file and more lerobot support

File: forked_cortex/gen3_lite_2f_macro.xacro (robot description, xacro)
@@ -15,25 +15,24 @@
   <xacro:if value="${use_fake_hardware or sim_isaac or sim_gazebo}">
     <xacro:unless value="${moveit_active}">
-    <!-- ros2 control include — skip for sim_gazebo because the gripper joint
-         is merged into the arm's GazeboSimSystem block instead (a separate
-         GripperHardwareInterface GazeboSimSystem instance cannot command joints). -->
-      <xacro:unless value="${sim_gazebo}">
-        <xacro:include filename="$(find kortex_description)/grippers/gen3_lite_2f/urdf/gen3_lite_2f.ros2_control.xacro" />
-        <xacro:if value="${use_fake_hardware}">
-          <xacro:property name="ros2_control_name" value="GenericSystem"/>
-        </xacro:if>
-        <xacro:unless value="${use_fake_hardware}">
-          <xacro:property name="ros2_control_name" value="${prefix}KortexMultiInterfaceHardware"/>
-        </xacro:unless>
-        <xacro:gripper_ros2_control
-          prefix="${prefix}"
-          use_fake_hardware="${use_fake_hardware}"
-          fake_sensor_commands="${fake_sensor_commands}"
-          sim_gazebo="false"
-          sim_isaac="${sim_isaac}"
-          isaac_joint_commands="${isaac_joint_commands}"
-          isaac_joint_states="${isaac_joint_states}"
-          tf_prefix=""/>
+    <!-- ros2 control include -->
+      <xacro:include filename="$(find kortex_description)/grippers/gen3_lite_2f/urdf/gen3_lite_2f.ros2_control.xacro" />
+      <xacro:if value="${sim_gazebo}">
+        <xacro:property name="ros2_control_name" value="GazeboSimSystem"/>
+      </xacro:if>
+      <xacro:if value="${use_fake_hardware}">
+        <xacro:property name="ros2_control_name" value="GenericSystem"/>
+      </xacro:if>
+      <xacro:unless value="${use_fake_hardware or sim_gazebo}">
+        <xacro:property name="ros2_control_name" value="${prefix}KortexMultiInterfaceHardware"/>
       </xacro:unless>
+      <xacro:gripper_ros2_control
+        prefix="${prefix}"
+        use_fake_hardware="${use_fake_hardware}"
+        fake_sensor_commands="${fake_sensor_commands}"
+        sim_gazebo="${sim_gazebo}"
+        sim_isaac="${sim_isaac}"
+        isaac_joint_commands="${isaac_joint_commands}"
+        isaac_joint_states="${isaac_joint_states}"
+        tf_prefix=""/>
   <!-- Tool frame used by the arm -->
       <link name="${prefix}tool_frame"/>
@@ -106,6 +105,6 @@
         <child link="${prefix}right_finger_prox_link" />
         <axis xyz="0 0 -1" />
-        <limit lower="-0.1" upper="0.96" effort="200" velocity="2.0" />
-        <dynamics damping="0.01" friction="0.0"/>
+        <limit lower="-0.1" upper="0.96" effort="10" velocity="0.6" />
+        <dynamics damping="0.1" friction="1"/>
       </joint>
       <link name="${prefix}right_finger_dist_link">
@@ -172,6 +171,6 @@
         <child link="${prefix}left_finger_prox_link" />
         <axis xyz="0 0 1" />
-        <limit lower="-0.1" upper="0.96" effort="200" velocity="2.0" />
-        <dynamics damping="0.01" friction="0.0"/>
+        <limit lower="-0.1" upper="0.96" effort="10" velocity="0.6" />
+        <dynamics damping="0.1" friction="1"/>
         <mimic joint="${prefix}right_finger_bottom_joint" multiplier="1.0" offset="0.0" />
       </joint>
@@ -284,5 +283,8 @@
         <child link="${prefix}right_finger_prox_link" />
         <axis xyz="0 0 -1" />
-        <limit lower="0.0" upper="0.85" effort="50" velocity="0.6" />
+        <!-- lower was 0.0; the real gripper's fully-open position overshoots to
+             ~-0.009 rad, which trips the ros2_control joint limiter and deactivates
+             the gripper controller. Small negative slack keeps it alive. -->
+        <limit lower="-0.02" upper="0.85" effort="50" velocity="0.6" />
       </joint>
       <link name="${prefix}right_finger_dist_link">
